File: eagle/trx-mainboard.sch (EAGLE design)
At the start: 11 parts, among them J1 629722000214

Commit message: Added display pinheader
Parts:
- added JP1: (no value), pinhead2:PINHD-1X08_2.54-SMD
Changed lines of the file:
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@@
 <part name="U$9" library="ai-thinker" library_urn="urn:adsk.eagle:library:18697339" deviceset="RA-02" device="" package3d_urn="urn:adsk.eagle:package:18697343/2"/>
 <part name="U$10" library="st-microelectronics" library_urn="urn:adsk.eagle:library:18661622" deviceset="STM32-F042X4/6-48" device="" package3d_urn="urn:adsk.eagle:package:18661624/3"/>
+<part name="JP1" library="pinhead2" library_urn="urn:adsk.eagle:library:40219860" deviceset="PINHD-1X08" device="_2.54-SMD" package3d_urn="urn:adsk.eagle:package:40220540/2"/>
 </parts>
 <sheets>
@@
 <instance part="U$9" gate="G$1" x="27.94" y="157.48" smashed="yes"/>
 <instance part="U$10" gate="G$1" x="116.84" y="157.48" smashed="yes"/>
+<instance part="JP1" gate="A" x="25.4" y="114.3" smashed="yes">
+<attribute name="NAME" x="19.05" y="127.635" size="1.778" layer="95"/>
+<attribute name="VALUE" x="19.05" y="101.6" size="1.778" layer="96"/>
+</instance>
 </instances>
 <busses>

Commit message: Added further components to pcb
Parts:
- added C1, C11, C12, C13, C2, C3: 100nF, rcl:C-EUC0805
- added C10, C4, C5, C6, C8: 4.7uF, rcl:C-EUC0805
- added C7: 1uF, rcl:C-EUC0805
- added C9: (no value), rcl:CPOL-EUC
- added R1, R2: 5.1k, rcl:R-EU_R0805
- added R3, R4, R5, R6: 3k, rcl:R-EU_R0805
- U$3: value BQ27441 -> BQ2407X; device texas-instruments:BQ27441 -> texas-instruments:BQ2407X
- U$4: value BQ2407X -> IHLP-1212; device texas-instruments:BQ2407X -> inductor-vishay:IHLP-1212
- U$6: value E22-900M30S -> E32-900M30S; device ebyte:E22-900M30S -> ebyte:E32-900M30S
Connections:
- new net +3V3: C1.1, C10.1, C13.1, C2.1, C3.1, C4.1, C8.1, C9.+, R6.1, U$10.VDD, U$10.VDDA, U$2.VOS, U$4.2, U$6.VCC, U$9.VDD
- new net BT_RX: U$10.PA2
- new net BT_TX: U$10.PA3
- new net GND: C1.2, C10.2, C11.2, C12.2, C13.2, C2.2, C3.2, C4.2, C5.2, C6.2, C7.2, C8.2, C9.-, R3.1, R4.1, R5.2, U$10.VSS, U$10.VSSA, U$2.DEV, U$2.FSW, U$3.!CE, U$3.EN2, U$3.SYSOFF, U$3.TMR, U$3.VSS, U$6.GND, U$8.1, U$9.VSS
- new net GPS_RX: U$10.PA9
- new net GPS_TX: U$10.PA10
- new net LORA1_D0: U$10.PA15, U$9.DIO0
- new net LORA1_MISO: U$10.PA6, U$9.MISO
- new net LORA1_MOSI: U$10.PA7, U$9.MOSI
- new net LORA1_RST: U$10.PA4, U$9.RESET
- new net LORA1_SCK: U$10.PA5, U$9.SCK
- new net LORA1_SSEL: U$10.PA8, U$9.NSS
- new net LORA2_D0: U$10.PB11, U$6.DIO0
- new net LORA2_MISO: U$10.PB14, U$6.MISO
- new net LORA2_MOSI: U$10.PB15, U$6.MOSI
- new net LORA2_RST: U$10.PB12, U$6.NRST
- new net LORA2_RXEN: U$10.PB9, U$6.RXEN
- new net LORA2_SCK: U$10.PB10, U$6.SCK
- new net LORA2_SSEL: U$10.PB13, U$6.NSS
- new net LORA2_TXEN: U$10.PB8, U$6.TXEN
- new net N$1: J1.CC1@1, R2.2
- new net N$10: U$2.AGND, U$2.FB, U$2.PGND
- new net N$2: J1.CC1@2, R1.2
- new net N$3: R3.2, U$3.ILM
- new net N$4: R4.2, U$3.ISET
- new net N$5: R5.1, U$3.TS
- new net N$6: U$2.SW, U$4.1
- new net N$7: C12.1, U$2.SS/TR
- new net N$8: R6.2, U$2.PG
- new net SWCLK: U$10.PA14
- new net SWDIO: U$10.PA13
- new net USB_D+: J1.D+1, J1.D+2, U$7.3
- new net USB_D-: J1.D-1, J1.D-2, U$7.2
- new net USB_DM: U$10.PA11, U$8.2
- new net USB_DP: U$10.PA12, U$8.3
- new net USB_GND: J1.GND, J1.GND1, J1.GND2, J1.GND3, J1.SHIELD, R1.1, R2.1, U$7.1
- new net USB_V: J1.VBUS, J1.VBUS1, J1.VBUS2, J1.VBUS3, U$7.4
- new net V+: C11.1, C5.1, U$2.AVIN, U$2.EN, U$2.PVIN, U$3.EN1, U$3.OUT
- new net VBAT+: C6.1, U$3.BAT
- new net VUSB: C7.1, U$3.IN, U$8.4
